Commit message: Added xacro

File: humblebot_description/urdf/humblebot.urdf (robot description, URDF)
Before this commit: robot humblebot, 41 links, 40 joints
Joints:
- joint base_wheel180_joint: origin xyz=0.060 -0.103 0 rpy=1.04 1.57 0 -> xyz=0.06 -0.10392304845413262 0 rpy=1.04 1.5707963267948966 0
- joint base_wheel300_joint: origin xyz=-0.12 0 0 rpy=0 1.57 3.14 -> xyz=-0.12 0.0 0 rpy=0 1.5707963267948966 3.141592653589793
- joint base_wheel60_joint: origin xyz=0.060 0.103 0 rpy=-1.04 1.57 0 -> xyz=0.06 0.10392304845413262 0 rpy=-1.0471975511965976 1.5707963267948966 0
- joint wheel_180deg_roller_1: origin xyz=0.035 0 0 rpy=1.57 0 0 -> xyz=0.035 0 0 rpy=1.5707963267948966 0 0
- joint wheel_180deg_roller_10: origin xyz=0.030 0.0175 0.030 rpy=1.57 0 0.57 -> xyz=0.03 0.0175 0.03 rpy=1.5707963267948966 0 0.57
- joint wheel_180deg_roller_11: origin xyz=-0.030 0.0175 0.030 rpy=1.57 0 -0.57 -> xyz=-0.03 0.0175 0.03 rpy=1.5707963267948966 0 -0.57
- joint wheel_180deg_roller_12: origin xyz=0.030 -0.0175 0.030 rpy=1.57 0 -0.57 -> xyz=0.03 -0.0175 0.03 rpy=1.5707963267948966 0 -0.57
- joint wheel_180deg_roller_2: origin xyz=-0.035 0 0 rpy=1.57 0 0 -> xyz=-0.035 0 0 rpy=1.5707963267948966 0 0
- joint wheel_180deg_roller_3: origin xyz=-0.0175 0.030 0 rpy=1.57 0 -1.047 -> xyz=-0.0175 0.03 0 rpy=1.5707963267948966 0 -1.0471975511965976
- joint wheel_180deg_roller_4: origin xyz=0.0175 -0.030 0 rpy=1.57 0 -1.047 -> xyz=0.0175 -0.03 0 rpy=1.5707963267948966 0 -1.0471975511965976
- joint wheel_180deg_roller_5: origin xyz=-0.0175 -0.030 0 rpy=1.57 0 1.047 -> xyz=-0.0175 -0.03 0 rpy=1.5707963267948966 0 1.0471975511965976
- joint wheel_180deg_roller_6: origin xyz=0.0175 0.030 0 rpy=1.57 0 1.047 -> xyz=0.0175 0.03 0 rpy=1.5707963267948966 0 1.0471975511965976
- joint wheel_180deg_roller_7: origin xyz=0 0.035 0.030 rpy=1.57 0 1.57 -> xyz=0 0.035 0.03 rpy=1.5707963267948966 0 1.5707963267948966
- joint wheel_180deg_roller_8: origin xyz=0 -0.035 0.030 rpy=1.57 0 1.57 -> xyz=0 -0.035 0.03 rpy=1.5707963267948966 0 1.5707963267948966
- joint wheel_180deg_roller_9: origin xyz=-0.030 -0.0175 0.030 rpy=1.57 0 0.57 -> xyz=-0.03 -0.0175 0.03 rpy=1.5707963267948966 0 0.57
- joint wheel_300deg_roller_1: origin xyz=0.035 0 0 rpy=1.57 0 0 -> xyz=0.035 0 0 rpy=1.5707963267948966 0 0
- joint wheel_300deg_roller_10: origin xyz=0.030 0.0175 0.030 rpy=1.57 0 0.57 -> xyz=0.03 0.0175 0.03 rpy=1.5707963267948966 0 0.57
- joint wheel_300deg_roller_11: origin xyz=-0.030 0.0175 0.030 rpy=1.57 0 -0.57 -> xyz=-0.03 0.0175 0.03 rpy=1.5707963267948966 0 -0.57
- joint wheel_300deg_roller_12: origin xyz=0.030 -0.0175 0.030 rpy=1.57 0 -0.57 -> xyz=0.03 -0.0175 0.03 rpy=1.5707963267948966 0 -0.57
- joint wheel_300deg_roller_2: origin xyz=-0.035 0 0 rpy=1.57 0 0 -> xyz=-0.035 0 0 rpy=1.5707963267948966 0 0
- joint wheel_300deg_roller_3: origin xyz=-0.0175 0.030 0 rpy=1.57 0 -1.047 -> xyz=-0.0175 0.03 0 rpy=1.5707963267948966 0 -1.0471975511965976
- joint wheel_300deg_roller_4: origin xyz=0.0175 -0.030 0 rpy=1.57 0 -1.047 -> xyz=0.0175 -0.03 0 rpy=1.5707963267948966 0 -1.0471975511965976
- joint wheel_300deg_roller_5: origin xyz=-0.0175 -0.030 0 rpy=1.57 0 1.047 -> xyz=-0.0175 -0.03 0 rpy=1.5707963267948966 0 1.0471975511965976
- joint wheel_300deg_roller_6: origin xyz=0.0175 0.030 0 rpy=1.57 0 1.047 -> xyz=0.0175 0.03 0 rpy=1.5707963267948966 0 1.0471975511965976
- joint wheel_300deg_roller_7: origin xyz=0 0.035 0.030 rpy=1.57 0 1.57 -> xyz=0 0.035 0.03 rpy=1.5707963267948966 0 1.5707963267948966
- joint wheel_300deg_roller_8: origin xyz=0 -0.035 0.030 rpy=1.57 0 1.57 -> xyz=0 -0.035 0.03 rpy=1.5707963267948966 0 1.5707963267948966
- joint wheel_300deg_roller_9: origin xyz=-0.030 -0.0175 0.030 rpy=1.57 0 0.57 -> xyz=-0.03 -0.0175 0.03 rpy=1.5707963267948966 0 0.57
- joint wheel_60deg_roller_1: origin xyz=0.035 0 0 rpy=1.57 0 0 -> xyz=0.035 0 0 rpy=1.5707963267948966 0 0
- joint wheel_60deg_roller_10: origin xyz=0.030 0.0175 0.030 rpy=1.57 0 0.57 -> xyz=0.03 0.0175 0.03 rpy=1.5707963267948966 0 0.57
- joint wheel_60deg_roller_11: origin xyz=-0.030 0.0175 0.030 rpy=1.57 0 -0.57 -> xyz=-0.03 0.0175 0.03 rpy=1.5707963267948966 0 -0.57
- joint wheel_60deg_roller_12: origin xyz=0.030 -0.0175 0.030 rpy=1.57 0 -0.57 -> xyz=0.03 -0.0175 0.03 rpy=1.5707963267948966 0 -0.57
- joint wheel_60deg_roller_2: origin xyz=-0.035 0 0 rpy=1.57 0 0 -> xyz=-0.035 0 0 rpy=1.5707963267948966 0 0
- joint wheel_60deg_roller_3: origin xyz=-0.0175 0.030 0 rpy=1.57 0 -1.047 -> xyz=-0.0175 0.03 0 rpy=1.5707963267948966 0 -1.0471975511965976
- joint wheel_60deg_roller_4: origin xyz=0.0175 -0.030 0 rpy=1.57 0 -1.047 -> xyz=0.0175 -0.03 0 rpy=1.5707963267948966 0 -1.0471975511965976
- joint wheel_60deg_roller_5: origin xyz=-0.0175 -0.030 0 rpy=1.57 0 1.047 -> xyz=-0.0175 -0.03 0 rpy=1.5707963267948966 0 1.0471975511965976
- joint wheel_60deg_roller_6: origin xyz=0.0175 0.030 0 rpy=1.57 0 1.047 -> xyz=0.0175 0.03 0 rpy=1.5707963267948966 0 1.0471975511965976
- joint wheel_60deg_roller_7: origin xyz=0 0.035 0.030 rpy=1.57 0 1.57 -> xyz=0 0.035 0.03 rpy=1.5707963267948966 0 1.5707963267948966
- joint wheel_60deg_roller_8: origin xyz=0 -0.035 0.030 rpy=1.57 0 1.57 -> xyz=0 -0.035 0.03 rpy=1.5707963267948966 0 1.5707963267948966
- joint wheel_60deg_roller_9: origin xyz=-0.030 -0.0175 0.030 rpy=1.57 0 0.57 -> xyz=-0.03 -0.0175 0.03 rpy=1.5707963267948966 0 0.57

Commit message: xacro update & Gazebo launch

File: humblebot_description/urdf/humblebot.urdf (robot description, URDF)
Before this commit: robot humblebot, 41 links, 40 joints
Links:
- link base_link: mass None -> 0.3; geometry collision cylinder length=0.08 radius=0.12; visual cylinder length=0.08 radius=0.12
- link wheel_180deg: mass None -> 0.02; geometry collision cylinder length=0.03 radius=0.035; visual cylinder length=0.03 radius=0.035
- link wheel_180deg_roller_1: mass None -> 0.003; geometry collision cylinder length=0.022 radius=0.0075; visual cylinder length=0.022 radius=0.0075
- link wheel_180deg_roller_10: mass None -> 0.003; geometry collision cylinder length=0.022 radius=0.0075; visual cylinder length=0.022 radius=0.0075
- link wheel_180deg_roller_11: mass None -> 0.003; geometry collision cylinder length=0.022 radius=0.0075; visual cylinder length=0.022 radius=0.0075
- link wheel_180deg_roller_12: mass None -> 0.003; geometry collision cylinder length=0.022 radius=0.0075; visual cylinder length=0.022 radius=0.0075
- link wheel_180deg_roller_2: mass None -> 0.003; geometry collision cylinder length=0.022 radius=0.0075; visual cylinder length=0.022 radius=0.0075
- link wheel_180deg_roller_3: mass None -> 0.003; geometry collision cylinder length=0.022 radius=0.0075; visual cylinder length=0.022 radius=0.0075
- link wheel_180deg_roller_4: mass None -> 0.003; geometry collision cylinder length=0.022 radius=0.0075; visual cylinder length=0.022 radius=0.0075
- link wheel_180deg_roller_5: mass None -> 0.003; geometry collision cylinder length=0.022 radius=0.0075; visual cylinder length=0.022 radius=0.0075
- link wheel_180deg_roller_6: mass None -> 0.003; geometry collision cylinder length=0.022 radius=0.0075; visual cylinder length=0.022 radius=0.0075
- link wheel_180deg_roller_7: mass None -> 0.003; geometry collision cylinder length=0.022 radius=0.0075; visual cylinder length=0.022 radius=0.0075
- link wheel_180deg_roller_8: mass None -> 0.003; geometry collision cylinder length=0.022 radius=0.0075; visual cylinder length=0.022 radius=0.0075
- link wheel_180deg_roller_9: mass None -> 0.003; geometry collision cylinder length=0.022 radius=0.0075; visual cylinder length=0.022 radius=0.0075
- link wheel_300deg: mass None -> 0.02; geometry collision cylinder length=0.03 radius=0.035; visual cylinder length=0.03 radius=0.035
- link wheel_300deg_roller_1: mass None -> 0.003; geometry collision cylinder length=0.022 radius=0.0075; visual cylinder length=0.022 radius=0.0075
- link wheel_300deg_roller_10: mass None -> 0.003; geometry collision cylinder length=0.022 radius=0.0075; visual cylinder length=0.022 radius=0.0075
- link wheel_300deg_roller_11: mass None -> 0.003; geometry collision cylinder length=0.022 radius=0.0075; visual cylinder length=0.022 radius=0.0075
- link wheel_300deg_roller_12: mass None -> 0.003; geometry collision cylinder length=0.022 radius=0.0075; visual cylinder length=0.022 radius=0.0075
- link wheel_300deg_roller_2: mass None -> 0.003; geometry collision cylinder length=0.022 radius=0.0075; visual cylinder length=0.022 radius=0.0075
- link wheel_300deg_roller_3: mass None -> 0.003; geometry collision cylinder length=0.022 radius=0.0075; visual cylinder length=0.022 radius=0.0075
- link wheel_300deg_roller_4: mass None -> 0.003; geometry collision cylinder length=0.022 radius=0.0075; visual cylinder length=0.022 radius=0.0075
- link wheel_300deg_roller_5: mass None -> 0.003; geometry collision cylinder length=0.022 radius=0.0075; visual cylinder length=0.022 radius=0.0075
- link wheel_300deg_roller_6: mass None -> 0.003; geometry collision cylinder length=0.022 radius=0.0075; visual cylinder length=0.022 radius=0.0075
- link wheel_300deg_roller_7: mass None -> 0.003; geometry collision cylinder length=0.022 radius=0.0075; visual cylinder length=0.022 radius=0.0075
- link wheel_300deg_roller_8: mass None -> 0.003; geometry collision cylinder length=0.022 radius=0.0075; visual cylinder length=0.022 radius=0.0075
- link wheel_300deg_roller_9: mass None -> 0.003; geometry collision cylinder length=0.022 radius=0.0075; visual cylinder length=0.022 radius=0.0075
- link wheel_60deg: mass None -> 0.02; geometry collision cylinder length=0.03 radius=0.035; visual cylinder length=0.03 radius=0.035
- link wheel_60deg_roller_1: mass None -> 0.003; geometry collision cylinder length=0.022 radius=0.0075; visual cylinder length=0.022 radius=0.0075
- link wheel_60deg_roller_10: mass None -> 0.003; geometry collision cylinder length=0.022 radius=0.0075; visual cylinder length=0.022 radius=0.0075
- link wheel_60deg_roller_11: mass None -> 0.003; geometry collision cylinder length=0.022 radius=0.0075; visual cylinder length=0.022 radius=0.0075
- link wheel_60deg_roller_12: mass None -> 0.003; geometry collision cylinder length=0.022 radius=0.0075; visual cylinder length=0.022 radius=0.0075
- link wheel_60deg_roller_2: mass None -> 0.003; geometry collision cylinder length=0.022 radius=0.0075; visual cylinder length=0.022 radius=0.0075
- link wheel_60deg_roller_3: mass None -> 0.003; geometry collision cylinder length=0.022 radius=0.0075; visual cylinder length=0.022 radius=0.0075
- link wheel_60deg_roller_4: mass None -> 0.003; geometry collision cylinder length=0.022 radius=0.0075; visual cylinder length=0.022 radius=0.0075
- link wheel_60deg_roller_5: mass None -> 0.003; geometry collision cylinder length=0.022 radius=0.0075; visual cylinder length=0.022 radius=0.0075
- link wheel_60deg_roller_6: mass None -> 0.003; geometry collision cylinder length=0.022 radius=0.0075; visual cylinder length=0.022 radius=0.0075
- link wheel_60deg_roller_7: mass None -> 0.003; geometry collision cylinder length=0.022 radius=0.0075; visual cylinder length=0.022 radius=0.0075
- link wheel_60deg_roller_8: mass None -> 0.003; geometry collision cylinder length=0.022 radius=0.0075; visual cylinder length=0.022 radius=0.0075
- link wheel_60deg_roller_9: mass None -> 0.003; geometry collision cylinder length=0.022 radius=0.0075; visual cylinder length=0.022 radius=0.0075
Joints:
- removed joint wheel_180deg_roller_1
- removed joint wheel_180deg_roller_10
- removed joint wheel_180deg_roller_11
- removed joint wheel_180deg_roller_12
- removed joint wheel_180deg_roller_2
- removed joint wheel_180deg_roller_3
- removed joint wheel_180deg_roller_4
- removed joint wheel_180deg_roller_5
- removed joint wheel_180deg_roller_6
- removed joint wheel_180deg_roller_7
- removed joint wheel_180deg_roller_8
- removed joint wheel_180deg_roller_9
- removed joint wheel_300deg_roller_1
- removed joint wheel_300deg_roller_10
- removed joint wheel_300deg_roller_11
- removed joint wheel_300deg_roller_12
- removed joint wheel_300deg_roller_2
- removed joint wheel_300deg_roller_3
- removed joint wheel_300deg_roller_4
- removed joint wheel_300deg_roller_5
- removed joint wheel_300deg_roller_6
- removed joint wheel_300deg_roller_7
- removed joint wheel_300deg_roller_8
- removed joint wheel_300deg_roller_9
- removed joint wheel_60deg_roller_1
- removed joint wheel_60deg_roller_10
- removed joint wheel_60deg_roller_11
- removed joint wheel_60deg_roller_12
- removed joint wheel_60deg_roller_2
- removed joint wheel_60deg_roller_3
- removed joint wheel_60deg_roller_4
- removed joint wheel_60deg_roller_5
- removed joint wheel_60deg_roller_6
- removed joint wheel_60deg_roller_7
- removed joint wheel_60deg_roller_8
- removed joint wheel_60deg_roller_9
- added joint wheel_180deg_roller_10_joint: type continuous, parent wheel_180deg, child wheel_180deg_roller_10, origin xyz=0.03 0.0175 0.03 rpy=1.5707963267948966 0 0.57, axis 0 0 1
- added joint wheel_180deg_roller_11_joint: type continuous, parent wheel_180deg, child wheel_180deg_roller_11, origin xyz=-0.03 0.0175 0.03 rpy=1.5707963267948966 0 -0.57, axis 0 0 1
- added joint wheel_180deg_roller_12_joint: type continuous, parent wheel_180deg, child wheel_180deg_roller_12, origin xyz=0.03 -0.0175 0.03 rpy=1.5707963267948966 0 -0.57, axis 0 0 1
- added joint wheel_180deg_roller_1_joint: type continuous, parent wheel_180deg, child wheel_180deg_roller_1, origin xyz=0.035 0 0 rpy=1.5707963267948966 0 0, axis 0 0 1
- added joint wheel_180deg_roller_2_joint: type continuous, parent wheel_180deg, child wheel_180deg_roller_2, origin xyz=-0.035 0 0 rpy=1.5707963267948966 0 0, axis 0 0 1
- added joint wheel_180deg_roller_3_joint: type continuous, parent wheel_180deg, child wheel_180deg_roller_3, origin xyz=-0.0175 0.03 0 rpy=1.5707963267948966 0 -1.0471975511965976, axis 0 0 1
- added joint wheel_180deg_roller_4_joint: type continuous, parent wheel_180deg, child wheel_180deg_roller_4, origin xyz=0.0175 -0.03 0 rpy=1.5707963267948966 0 -1.0471975511965976, axis 0 0 1
- added joint wheel_180deg_roller_5_joint: type continuous, parent wheel_180deg, child wheel_180deg_roller_5, origin xyz=-0.0175 -0.03 0 rpy=1.5707963267948966 0 1.0471975511965976, axis 0 0 1
- added joint wheel_180deg_roller_6_joint: type continuous, parent wheel_180deg, child wheel_180deg_roller_6, origin xyz=0.0175 0.03 0 rpy=1.5707963267948966 0 1.0471975511965976, axis 0 0 1
- added joint wheel_180deg_roller_7_joint: type continuous, parent wheel_180deg, child wheel_180deg_roller_7, origin xyz=0 0.035 0.03 rpy=1.5707963267948966 0 1.5707963267948966, axis 0 0 1
- added joint wheel_180deg_roller_8_joint: type continuous, parent wheel_180deg, child wheel_180deg_roller_8, origin xyz=0 -0.035 0.03 rpy=1.5707963267948966 0 1.5707963267948966, axis 0 0 1
- added joint wheel_180deg_roller_9_joint: type continuous, parent wheel_180deg, child wheel_180deg_roller_9, origin xyz=-0.03 -0.0175 0.03 rpy=1.5707963267948966 0 0.57, axis 0 0 1
- added joint wheel_300deg_roller_10_joint: type continuous, parent wheel_300deg, child wheel_300deg_roller_10, origin xyz=0.03 0.0175 0.03 rpy=1.5707963267948966 0 0.57, axis 0 0 1
- added joint wheel_300deg_roller_11_joint: type continuous, parent wheel_300deg, child wheel_300deg_roller_11, origin xyz=-0.03 0.0175 0.03 rpy=1.5707963267948966 0 -0.57, axis 0 0 1
- added joint wheel_300deg_roller_12_joint: type continuous, parent wheel_300deg, child wheel_300deg_roller_12, origin xyz=0.03 -0.0175 0.03 rpy=1.5707963267948966 0 -0.57, axis 0 0 1
- added joint wheel_300deg_roller_1_joint: type continuous, parent wheel_300deg, child wheel_300deg_roller_1, origin xyz=0.035 0 0 rpy=1.5707963267948966 0 0, axis 0 0 1
- added joint wheel_300deg_roller_2_joint: type continuous, parent wheel_300deg, child wheel_300deg_roller_2, origin xyz=-0.035 0 0 rpy=1.5707963267948966 0 0, axis 0 0 1
- added joint wheel_300deg_roller_3_joint: type continuous, parent wheel_300deg, child wheel_300deg_roller_3, origin xyz=-0.0175 0.03 0 rpy=1.5707963267948966 0 -1.0471975511965976, axis 0 0 1
- added joint wheel_300deg_roller_4_joint: type continuous, parent wheel_300deg, child wheel_300deg_roller_4, origin xyz=0.0175 -0.03 0 rpy=1.5707963267948966 0 -1.0471975511965976, axis 0 0 1
- added joint wheel_300deg_roller_5_joint: type continuous, parent wheel_300deg, child wheel_300deg_roller_5, origin xyz=-0.0175 -0.03 0 rpy=1.5707963267948966 0 1.0471975511965976, axis 0 0 1
- added joint wheel_300deg_roller_6_joint: type continuous, parent wheel_300deg, child wheel_300deg_roller_6, origin xyz=0.0175 0.03 0 rpy=1.5707963267948966 0 1.0471975511965976, axis 0 0 1
- added joint wheel_300deg_roller_7_joint: type continuous, parent wheel_300deg, child wheel_300deg_roller_7, origin xyz=0 0.035 0.03 rpy=1.5707963267948966 0 1.5707963267948966, axis 0 0 1
- added joint wheel_300deg_roller_8_joint: type continuous, parent wheel_300deg, child wheel_300deg_roller_8, origin xyz=0 -0.035 0.03 rpy=1.5707963267948966 0 1.5707963267948966, axis 0 0 1
- added joint wheel_300deg_roller_9_joint: type continuous, parent wheel_300deg, child wheel_300deg_roller_9, origin xyz=-0.03 -0.0175 0.03 rpy=1.5707963267948966 0 0.57, axis 0 0 1
- added joint wheel_60deg_roller_10_joint: type continuous, parent wheel_60deg, child wheel_60deg_roller_10, origin xyz=0.03 0.0175 0.03 rpy=1.5707963267948966 0 0.57, axis 0 0 1
- added joint wheel_60deg_roller_11_joint: type continuous, parent wheel_60deg, child wheel_60deg_roller_11, origin xyz=-0.03 0.0175 0.03 rpy=1.5707963267948966 0 -0.57, axis 0 0 1
- added joint wheel_60deg_roller_12_joint: type continuous, parent wheel_60deg, child wheel_60deg_roller_12, origin xyz=0.03 -0.0175 0.03 rpy=1.5707963267948966 0 -0.57, axis 0 0 1
- added joint wheel_60deg_roller_1_joint: type continuous, parent wheel_60deg, child wheel_60deg_roller_1, origin xyz=0.035 0 0 rpy=1.5707963267948966 0 0, axis 0 0 1
- added joint wheel_60deg_roller_2_joint: type continuous, parent wheel_60deg, child wheel_60deg_roller_2, origin xyz=-0.035 0 0 rpy=1.5707963267948966 0 0, axis 0 0 1
- added joint wheel_60deg_roller_3_joint: type continuous, parent wheel_60deg, child wheel_60deg_roller_3, origin xyz=-0.0175 0.03 0 rpy=1.5707963267948966 0 -1.0471975511965976, axis 0 0 1
- added joint wheel_60deg_roller_4_joint: type continuous, parent wheel_60deg, child wheel_60deg_roller_4, origin xyz=0.0175 -0.03 0 rpy=1.5707963267948966 0 -1.0471975511965976, axis 0 0 1
- added joint wheel_60deg_roller_5_joint: type continuous, parent wheel_60deg, child wheel_60deg_roller_5, origin xyz=-0.0175 -0.03 0 rpy=1.5707963267948966 0 1.0471975511965976, axis 0 0 1
- added joint wheel_60deg_roller_6_joint: type continuous, parent wheel_60deg, child wheel_60deg_roller_6, origin xyz=0.0175 0.03 0 rpy=1.5707963267948966 0 1.0471975511965976, axis 0 0 1
- added joint wheel_60deg_roller_7_joint: type continuous, parent wheel_60deg, child wheel_60deg_roller_7, origin xyz=0 0.035 0.03 rpy=1.5707963267948966 0 1.5707963267948966, axis 0 0 1
- added joint wheel_60deg_roller_8_joint: type continuous, parent wheel_60deg, child wheel_60deg_roller_8, origin xyz=0 -0.035 0.03 rpy=1.5707963267948966 0 1.5707963267948966, axis 0 0 1
- added joint wheel_60deg_roller_9_joint: type continuous, parent wheel_60deg, child wheel_60deg_roller_9, origin xyz=-0.03 -0.0175 0.03 rpy=1.5707963267948966 0 0.57, axis 0 0 1
