Commit message: xacro update & Gazebo launch

File: humblebot_description/urdf/humblebot.xacro (robot description, xacro)
@@ -1,636 +1,7 @@
 <?xml version="1.0"?>
 <robot name="humblebot" xmlns:xacro="http://www.ros.org/wiki/xacro">
-    <xacro:property name="base_radius" value="0.12" />
-    <xacro:property name="base_length" value="0.08" />
-    <xacro:property name="wheel_radius" value="0.035" />
-    <xacro:property name="wheel_length" value="0.03" />
-    <xacro:property name="roller_radius" value="0.0075" />
-    <xacro:property name="roller_length" value="0.022" />
-    <!-- derived/utility properties used in origin formulas -->
-    <!-- 60 deg and -60 deg components -->
-    <xacro:property name="cos60" value="${0.5}" />
-    <xacro:property name="sin60" value="${0.8660254037844386}" />
-    <xacro:property name="cos_m60" value="${0.5}" />
-    <xacro:property name="sin_m60" value="${-0.8660254037844386}" />
-    <!-- 180 deg components -->
-    <xacro:property name="cos180" value="${-1.0}" />
-    <xacro:property name="sin180" value="${0.0}" />
-    <!-- wheel center positions (derived from base radius and angle) -->
-    <xacro:property name="wheel60_x" value="${base_radius * cos60}" />
-    <xacro:property name="wheel60_y" value="${base_radius * sin60}" />
-    <xacro:property name="wheel300_x" value="${base_radius * cos180}" />
-    <xacro:property name="wheel300_y" value="${base_radius * sin180}" />
-    <xacro:property name="wheel180_x" value="${base_radius * cos_m60}" />
-    <xacro:property name="wheel180_y" value="${base_radius * sin_m60}" />
-    <!-- some helper values used inside roller joint origins -->
-    <xacro:property name="half_wheel_radius" value="${wheel_radius / 2.0}" />
-    <material name="green">
-        <color rgba="0 1 0 1" />
-    </material>
-    <material name="black">
-        <color rgba="0 0 0 1" />
-    </material>
-    <link name="base_footprint" />
-    <link name="base_link">
-        <visual>
-            <geometry>
-                <cylinder radius="${base_radius}" length="${base_length}" />
-            </geometry>
-            <origin xyz="0 0 ${base_length / 2.0}" rpy="0 0 0" />
-            <material name="green" />
-        </visual>
-    </link>
-    <!--Wheel 60deg-->
-    <link name="wheel_60deg">
-        <visual>
-            <geometry>
-                <cylinder radius="${wheel_radius}" length="${wheel_length}" />
-            </geometry>
-            <origin xyz="0 0 ${wheel_length / 2.0}" rpy="0 0 0" />
-            <material name="green" />
-        </visual>
-    </link>
-    <link name="wheel_60deg_roller_1">
-        <visual>
-            <geometry>
-                <cylinder radius="${roller_radius}" length="${roller_length}" />
-            </geometry>
-            <origin xyz="0 0 0" rpy="0 0 0" />
-            <material name="black" />
-        </visual>
-    </link>
-    <link name="wheel_60deg_roller_2">
-        <visual>
-            <geometry>
-                <cylinder radius="${roller_radius}" length="${roller_length}" />
-            </geometry>
-            <origin xyz="0 0 0" rpy="0 0 0" />
-            <material name="black" />
-        </visual>
-    </link>
-    <link name="wheel_60deg_roller_3">
-        <visual>
-            <geometry>
-                <cylinder radius="${roller_radius}" length="${roller_length}" />
-            </geometry>
-            <origin xyz="0 0 0" rpy="0 0 0" />
-            <material name="black" />
-        </visual>
-    </link>
-    <link name="wheel_60deg_roller_4">
-        <visual>
-            <geometry>
-                <cylinder radius="${roller_radius}" length="${roller_length}" />
-            </geometry>
-            <origin xyz="0 0 0" rpy="0 0 0" />
-            <material name="black" />
-        </visual>
-    </link>
-    <link name="wheel_60deg_roller_5">
-        <visual>
-            <geometry>
-                <cylinder radius="${roller_radius}" length="${roller_length}" />
-            </geometry>
-            <origin xyz="0 0 0" rpy="0 0 0" />
-            <material name="black" />
-        </visual>
-    </link>
-    <link name="wheel_60deg_roller_6">
-        <visual>
-            <geometry>
-                <cylinder radius="${roller_radius}" length="${roller_length}" />
-            </geometry>
-            <origin xyz="0 0 0" rpy="0 0 0" />
-            <material name="black" />
-        </visual>
-    </link>
-    <link name="wheel_60deg_roller_7">
-        <visual>
-            <geometry>
-                <cylinder radius="${roller_radius}" length="${roller_length}" />
-            </geometry>
-            <origin xyz="0 0 0" rpy="0 0 0" />
-            <material name="black" />
-        </visual>
-    </link>
-    <link name="wheel_60deg_roller_8">
-        <visual>
-            <geometry>
-                <cylinder radius="${roller_radius}" length="${roller_length}" />
-            </geometry>
-            <origin xyz="0 0 0" rpy="0 0 0" />
-            <material name="black" />
-        </visual>
-    </link>
-    <link name="wheel_60deg_roller_9">
-        <visual>
-            <geometry>
-                <cylinder radius="${roller_radius}" length="${roller_length}" />
-            </geometry>
-            <origin xyz="0 0 0" rpy="0 0 0" />
-            <material name="black" />
-        </visual>
-    </link>
-    <link name="wheel_60deg_roller_10">
-        <visual>
-            <geometry>
-                <cylinder radius="${roller_radius}" length="${roller_length}" />
-            </geometry>
-            <origin xyz="0 0 0" rpy="0 0 0" />
-            <material name="black" />
-        </visual>
-    </link>
-    <link name="wheel_60deg_roller_11">
-        <visual>
-            <geometry>
-                <cylinder radius="${roller_radius}" length="${roller_length}" />
-            </geometry>
-            <origin xyz="0 0 0" rpy="0 0 0" />
-            <material name="black" />
-        </visual>
-    </link>
-    <link name="wheel_60deg_roller_12">
-        <visual>
-            <geometry>
-                <cylinder radius="${roller_radius}" length="${roller_length}" />
-            </geometry>
-            <origin xyz="0 0 0" rpy="0 0 0" />
-            <material name="black" />
-        </visual>
-    </link>
-    <joint name="base_joint" type="fixed">
-        <parent link="base_footprint" />
-        <child link="base_link" />
-        <origin xyz="0 0 ${wheel_radius}" rpy="0 0 0" />
-    </joint>
-    <joint name="base_wheel60_joint" type="continuous">
-        <parent link="base_link" />
-        <child link="wheel_60deg" />
-        <axis xyz="0 0 1" />
-        <origin xyz="${wheel60_x} ${wheel60_y} 0" rpy="${-pi / 3.0} ${pi / 2.0} 0" />
-    </joint>
-    <joint name="wheel_60deg_roller_1" type="continuous">
-        <parent link="wheel_60deg" />
-        <child link="wheel_60deg_roller_1" />
-        <axis xyz="0 0 1" />
-        <origin xyz="${wheel_radius} 0 0" rpy="${pi / 2.0} 0 0" />
-    </joint>
-    <joint name="wheel_60deg_roller_2" type="continuous">
-        <parent link="wheel_60deg" />
-        <child link="wheel_60deg_roller_2" />
-        <axis xyz="0 0 1" />
-        <origin xyz="-${wheel_radius} 0 0" rpy="${pi / 2.0} 0 0" />
-    </joint>
-    <joint name="wheel_60deg_roller_3" type="continuous">
-        <parent link="wheel_60deg" />
-        <child link="wheel_60deg_roller_3" />
-        <axis xyz="0 0 1" />
-        <origin xyz="-${half_wheel_radius} ${wheel_length} 0" rpy="${pi / 2.0} 0 ${-pi / 3.0}" />
-    </joint>
-    <joint name="wheel_60deg_roller_4" type="continuous">
-        <parent link="wheel_60deg" />
-        <child link="wheel_60deg_roller_4" />
-        <axis xyz="0 0 1" />
-        <origin xyz="${half_wheel_radius} -${wheel_length} 0" rpy="${pi / 2.0} 0 ${-pi / 3.0}" />
-    </joint>
-    <joint name="wheel_60deg_roller_5" type="continuous">
-        <parent link="wheel_60deg" />
-        <child link="wheel_60deg_roller_5" />
-        <axis xyz="0 0 1" />
-        <origin xyz="-${half_wheel_radius} -${wheel_length} 0" rpy="${pi / 2.0} 0 ${pi / 3.0}" />
-    </joint>
-    <joint name="wheel_60deg_roller_6" type="continuous">
-        <parent link="wheel_60deg" />
-        <child link="wheel_60deg_roller_6" />
-        <axis xyz="0 0 1" />
-        <origin xyz="${half_wheel_radius} ${wheel_length} 0" rpy="${pi / 2.0} 0 ${pi / 3.0}" />
-    </joint>
-    <joint name="wheel_60deg_roller_7" type="continuous">
-        <parent link="wheel_60deg" />
-        <child link="wheel_60deg_roller_7" />
-        <axis xyz="0 0 1" />
-        <origin xyz="0 ${wheel_radius} ${wheel_length}" rpy="${pi / 2.0} 0 ${pi / 2.0}" />
-    </joint>
-    <joint name="wheel_60deg_roller_8" type="continuous">
-        <parent link="wheel_60deg" />
-        <child link="wheel_60deg_roller_8" />
-        <axis xyz="0 0 1" />
-        <origin xyz="0 -${wheel_radius} ${wheel_length}" rpy="${pi / 2.0} 0 ${pi / 2.0}" />
-    </joint>
-    <joint name="wheel_60deg_roller_9" type="continuous">
-        <parent link="wheel_60deg" />
-        <child link="wheel_60deg_roller_9" />
-        <axis xyz="0 0 1" />
-        <origin xyz="-${wheel_length} -${half_wheel_radius} ${wheel_length}" rpy="${pi / 2.0} 0 0.57" />
-    </joint>
-    <joint name="wheel_60deg_roller_10" type="continuous">
-        <parent link="wheel_60deg" />
-        <child link="wheel_60deg_roller_10" />
-        <axis xyz="0 0 1" />
-        <origin xyz="${wheel_length} ${half_wheel_radius} ${wheel_length}" rpy="${pi / 2.0} 0 0.57" />
-    </joint>
-    <joint name="wheel_60deg_roller_11" type="continuous">
-        <parent link="wheel_60deg" />
-        <child link="wheel_60deg_roller_11" />
-        <axis xyz="0 0 1" />
-        <origin xyz="-${wheel_length} ${half_wheel_radius} ${wheel_length}" rpy="${pi / 2.0} 0 -0.57" />
-    </joint>
-    <joint name="wheel_60deg_roller_12" type="continuous">
-        <parent link="wheel_60deg" />
-        <child link="wheel_60deg_roller_12" />
-        <axis xyz="0 0 1" />
-        <origin xyz="${wheel_length} -${half_wheel_radius} ${wheel_length}" rpy="${pi / 2.0} 0 -0.57" />
-    </joint>
-    <!--Wheel 300deg-->
-    <link name="wheel_300deg">
-        <visual>
-            <geometry>
-                <cylinder radius="${wheel_radius}" length="${wheel_length}" />
-            </geometry>
-            <origin xyz="0 0 ${wheel_length / 2.0}" rpy="0 0 0" />
-            <material name="green" />
-        </visual>
-    </link>
-    <link name="wheel_300deg_roller_1">
-        <visual>
-            <geometry>
-                <cylinder radius="${roller_radius}" length="${roller_length}" />
-            </geometry>
-            <origin xyz="0 0 0" rpy="0 0 0" />
-            <material name="black" />
-        </visual>
-    </link>
-    <link name="wheel_300deg_roller_2">
-        <visual>
-            <geometry>
-                <cylinder radius="${roller_radius}" length="${roller_length}" />
-            </geometry>
-            <origin xyz="0 0 0" rpy="0 0 0" />
-            <material name="black" />
-        </visual>
-    </link>
-    <link name="wheel_300deg_roller_3">
-        <visual>
-            <geometry>
-                <cylinder radius="${roller_radius}" length="${roller_length}" />
-            </geometry>
-            <origin xyz="0 0 0" rpy="0 0 0" />
-            <material name="black" />
-        </visual>
-    </link>
-    <link name="wheel_300deg_roller_4">
-        <visual>
-            <geometry>
-                <cylinder radius="${roller_radius}" length="${roller_length}" />
-            </geometry>
-            <origin xyz="0 0 0" rpy="0 0 0" />
-            <material name="black" />
-        </visual>
-    </link>
-    <link name="wheel_300deg_roller_5">
-        <visual>
-            <geometry>
-                <cylinder radius="${roller_radius}" length="${roller_length}" />
-            </geometry>
-            <origin xyz="0 0 0" rpy="0 0 0" />
-            <material name="black" />
-        </visual>
-    </link>
-    <link name="wheel_300deg_roller_6">
-        <visual>
-            <geometry>
-                <cylinder radius="${roller_radius}" length="${roller_length}" />
-            </geometry>
-            <origin xyz="0 0 0" rpy="0 0 0" />
-            <material name="black" />
-        </visual>
-    </link>
-    <link name="wheel_300deg_roller_7">
-        <visual>
-            <geometry>
-                <cylinder radius="${roller_radius}" length="${roller_length}" />
-            </geometry>
-            <origin xyz="0 0 0" rpy="0 0 0" />
-            <material name="black" />
-        </visual>
-    </link>
-    <link name="wheel_300deg_roller_8">
-        <visual>
-            <geometry>
-                <cylinder radius="${roller_radius}" length="${roller_length}" />
-            </geometry>
-            <origin xyz="0 0 0" rpy="0 0 0" />
-            <material name="black" />
-        </visual>
-    </link>
-    <link name="wheel_300deg_roller_9">
-        <visual>
-            <geometry>
-                <cylinder radius="${roller_radius}" length="${roller_length}" />
-            </geometry>
-            <origin xyz="0 0 0" rpy="0 0 0" />
-            <material name="black" />
-        </visual>
-    </link>
-    <link name="wheel_300deg_roller_10">
-        <visual>
-            <geometry>
-                <cylinder radius="${roller_radius}" length="${roller_length}" />
-            </geometry>
-            <origin xyz="0 0 0" rpy="0 0 0" />
-            <material name="black" />
-        </visual>
-    </link>
-    <link name="wheel_300deg_roller_11">
-        <visual>
-            <geometry>
-                <cylinder radius="${roller_radius}" length="${roller_length}" />
-            </geometry>
-            <origin xyz="0 0 0" rpy="0 0 0" />
-            <material name="black" />
-        </visual>
-    </link>
-    <link name="wheel_300deg_roller_12">
-        <visual>
-            <geometry>
-                <cylinder radius="${roller_radius}" length="${roller_length}" />
-            </geometry>
-            <origin xyz="0 0 0" rpy="0 0 0" />
-            <material name="black" />
-        </visual>
-    </link>
-    <joint name="base_wheel300_joint" type="continuous">
-        <parent link="base_link" />
-        <child link="wheel_300deg" />
-        <axis xyz="0 0 1" />
-        <origin xyz="${wheel300_x} ${wheel300_y} 0" rpy="0 ${pi / 2.0} ${pi}" />
-    </joint>
-    <joint name="wheel_300deg_roller_1" type="continuous">
-        <parent link="wheel_300deg" />
-        <child link="wheel_300deg_roller_1" />
-        <axis xyz="0 0 1" />
-        <origin xyz="${wheel_radius} 0 0" rpy="${pi / 2.0} 0 0" />
-    </joint>
-    <joint name="wheel_300deg_roller_2" type="continuous">
-        <parent link="wheel_300deg" />
-        <child link="wheel_300deg_roller_2" />
-        <axis xyz="0 0 1" />
-        <origin xyz="-${wheel_radius} 0 0" rpy="${pi / 2.0} 0 0" />
-    </joint>
-    <joint name="wheel_300deg_roller_3" type="continuous">
-        <parent link="wheel_300deg" />
-        <child link="wheel_300deg_roller_3" />
-        <axis xyz="0 0 1" />
-        <origin xyz="-${half_wheel_radius} ${wheel_length} 0" rpy="${pi / 2.0} 0 ${-pi / 3.0}" />
-    </joint>
-    <joint name="wheel_300deg_roller_4" type="continuous">
-        <parent link="wheel_300deg" />
-        <child link="wheel_300deg_roller_4" />
-        <axis xyz="0 0 1" />
-        <origin xyz="${half_wheel_radius} -${wheel_length} 0" rpy="${pi / 2.0} 0 ${-pi / 3.0}" />
-    </joint>
-    <joint name="wheel_300deg_roller_5" type="continuous">
-        <parent link="wheel_300deg" />
-        <child link="wheel_300deg_roller_5" />
-        <axis xyz="0 0 1" />
-        <origin xyz="-${half_wheel_radius} -${wheel_length} 0" rpy="${pi / 2.0} 0 ${pi / 3.0}" />
-    </joint>
-    <joint name="wheel_300deg_roller_6" type="continuous">
-        <parent link="wheel_300deg" />
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